File: RAM card/ram-card-256k/ram-card-256k.kicad_pcb (KiCad board)
At the start: 2 copper layers, 41.9 x 54.1 mm, 12 parts, among them J1 RAM card connector, U1 HC138, U2 KM681000BLG, U3 KM681000BLG

Commit message: Assign 3d-model
Parts:
- U1: footprint Package_SO:SOP-16_3.9x9.9mm_P1.27mm -> Package_SO:SOIC-16_3.9x9.9mm_P1.27mm
Routing:
- net /A2: track 78.6 -> 79.9 mm
- net /A1: track 85.6 -> 86.9 mm
- net /A0: track 92.5 -> 93.7 mm

Commit message: Add README
Other:
- board text added: "read only"
Changed lines of the file:
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@@
       (effects (font (size 1 1) (thickness 0.15)))
     )
+    (fp_line (start -2.25 -1) (end 1.65 -1) (layer "F.SilkS") (width 0.12))
+    (fp_line (start -2.25 1) (end 1.65 1) (layer "F.SilkS") (width 0.12))
     (fp_line (start -2.25 -1) (end -2.25 1) (layer "F.SilkS") (width 0.12))
-    (fp_line (start -2.25 1) (end 1.65 1) (layer "F.SilkS") (width 0.12))
-    (fp_line (start -2.25 -1) (end 1.65 -1) (layer "F.SilkS") (width 0.12))
     (fp_line (start 2.35 -1.15) (end 2.35 1.15) (layer "F.CrtYd") (width 0.05))
     (fp_line (start -2.35 -1.15) (end -2.35 1.15) (layer "F.CrtYd") (width 0.05))
+    (fp_line (start -2.35 -1.15) (end 2.35 -1.15) (layer "F.CrtYd") (width 0.05))
     (fp_line (start 2.35 1.15) (end -2.35 1.15) (layer "F.CrtYd") (width 0.05))
-    (fp_line (start -2.35 -1.15) (end 2.35 -1.15) (layer "F.CrtYd") (width 0.05))
-    (fp_line (start 0.25 -0.4) (end 0.25 0.4) (layer "F.Fab") (width 0.1))
     (fp_line (start 1.4 0.9) (end -1.4 0.9) (layer "F.Fab") (width 0.1))
     (fp_line (start -0.35 0) (end -0.35 -0.55) (layer "F.Fab") (width 0.1))
-    (fp_line (start 0.25 0) (end 0.75 0) (layer "F.Fab") (width 0.1))
     (fp_line (start 0.25 0.4) (end -0.35 0) (layer "F.Fab") (width 0.1))
-    (fp_line (start -0.75 0) (end -0.35 0) (layer "F.Fab") (width 0.1))
+    (fp_line (start -1.4 -0.9) (end 1.4 -0.9) (layer "F.Fab") (width 0.1))
+    (fp_line (start -1.4 0.9) (end -1.4 -0.9) (layer "F.Fab") (width 0.1))
     (fp_line (start 1.4 -0.9) (end 1.4 0.9) (layer "F.Fab") (width 0.1))
     (fp_line (start -0.35 0) (end -0.35 0.55) (layer "F.Fab") (width 0.1))
+    (fp_line (start 0.25 0) (end 0.75 0) (layer "F.Fab") (width 0.1))
+    (fp_line (start 0.25 -0.4) (end 0.25 0.4) (layer "F.Fab") (width 0.1))
     (fp_line (start -0.35 0) (end 0.25 -0.4) (layer "F.Fab") (width 0.1))
-    (fp_line (start -1.4 0.9) (end -1.4 -0.9) (layer "F.Fab") (width 0.1))
-    (fp_line (start -1.4 -0.9) (end 1.4 -0.9) (layer "F.Fab") (width 0.1))
+    (fp_line (start -0.75 0) (end -0.35 0) (layer "F.Fab") (width 0.1))
     (pad "1" smd rect locked (at -1.65 0 90) (size 0.9 1.2) (layers "F.Cu" "F.Paste" "F.Mask")
       (net 3 "VCC") (pinfunction "K") (pintype "passive"))
@@
     (property "Sheetname" "")
     (attr smd)
-    (fp_text reference "J1" (at -1.27 25.4 180 unlocked) (layer "B.SilkS")
+    (fp_text reference "J1" (at -1.27 25.4 180 unlocked) (layer "B.SilkS") hide
       (effects (font (size 1 1) (thickness 0.15)) (justify mirror))
     )
@@
     (effects (font (size 1 1) (thickness 0.1524)))
   )
+  (gr_text "read\nonly" (at 127.508 52.324) (layer "F.SilkS")
+    (effects (font (size 0.8128 0.8128) (thickness 0.1524)))
+  )
   (segment (start 146.685 59.055) (end 146.685 60.58) (width 0.6) (layer "F.Cu") (net 1))
