File: casio-pb-2000/ROM-card/ROM-card-64K/ROM-card-64K.kicad_sch (KiCad schematic)
At the start: 2 parts, among them J1 casio_connector_45pins, U1 27C512PLCC

Commit message: Design footprint
Parts:
- J1: footprint (none) -> custom:ROM_card_connector_45
Changed lines of the file:
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@@
       (effects (font (size 1.27 1.27)) hide)
     )
-    (property "Footprint" "" (id 2) (at 44.45 29.21 0)
+    (property "Footprint" "custom:ROM_card_connector_45" (id 2) (at 44.45 29.21 0)
       (effects (font (size 1.27 1.27)) hide)
     )
@@
     )
     (path "/f3db7c4d-8e12-40af-a5c4-82758ab1f297"
-      (reference "J1") (unit 1) (value "casio_connector_45pins") (footprint "")
+      (reference "J1") (unit 1) (value "casio_connector_45pins") (footprint "custom:ROM_card_connector_45")
     )
     (path "/81f57ec5-39f7-4164-9845-5a54c0ccbe20"
